Commit message: feat: first grab ok

File: style3d/examples/franka_emika_panda/urdf/fr3_franka_hand_new.urdf (robot description, URDF)
Before this commit: robot fr3, 14 links, 13 joints
Links:
- link fr3_leftfinger: geometry collision mesh filename=package://franka_emika_panda/meshes/robot_ee/franka_hand_wh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; visual mesh filename=package://franka_emika_panda/meshes/robot_ee/franka_hand_wh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
- link fr3_rightfinger: geometry collision mesh filename=package://franka_emika_panda/meshes/robot_ee/franka_hand_wh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; visual mesh filename=package://franka_emika_panda/meshes/robot_ee/franka_hand_wh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

Commit message: feat: use_frozen_cloth with name convention

File: style3d/examples/franka_emika_panda/urdf/fr3_franka_hand_new.urdf (robot description, URDF)
Before this commit: robot fr3, 14 links, 13 joints
Links:
- removed link fr3_leftfinger
- removed link fr3_rightfinger
- added link fr3_leftfinger_s3d, mass 0.0291; collision mesh filename=package://franka_emika_panda/meshes/robot_ee/franka_hand_wh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; visual mesh filename=package://franka_emika_panda/meshes/robot_ee/franka_hand_wh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
- added link fr3_rightfinger_s3d, mass 0.0291; collision mesh filename=package://franka_emika_panda/meshes/robot_ee/franka_hand_wh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; visual mesh filename=package://franka_emika_panda/meshes/robot_ee/franka_hand_wh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
Joints:
- joint fr3_finger_joint1: child fr3_leftfinger -> fr3_leftfinger_s3d
- joint fr3_finger_joint2: child fr3_rightfinger -> fr3_rightfinger_s3d
